File: SatelitesPowerAmplifier.sch (KiCad schematic (older format))
At the start: 41 parts

Commit message: Change input cascade
Parts:
- removed Q? (x2): КТ808А, symbol Q_NPN_BCE
- removed R?: R, symbol R
- removed RV? (x2): POT, symbol POT
- added D? (x2): D, symbol D
- added Q? (x2): КТ808А, symbol Q_NPN_EBC
- added R? (x4): R, symbol R
- P?: value CONN_01X02 -> A/AB
- P?: value CONN_01X02 -> IN
- R? (x2): value R -> 43
Connections:
- wire segments 85 -> 124
Other:
- moved on the sheet: C?, D?, P?, Q?, R?

Commit message: Add DAC
Connections:
- wire segments 124 -> 85
Changed lines of the file:
@@
 LIBS:valves
 LIBS:tda7293v
+LIBS:ad1955
 LIBS:amplifier-cache
 EELAYER 26 0
@@
 	3550 4200 3550 4150
 Wire Wire Line
-	3450 4150 3550 4150
-Wire Wire Line
-	3550 4150 3600 4150
+	3450 4150 3600 4150
 Wire Wire Line
 	4850 4850 4850 4950
@@
 	3700 3400 3700 3450
 Wire Wire Line
-	3650 3400 3700 3400
-Wire Wire Line
-	3700 3400 4700 3400
+	3650 3400 4700 3400
 Wire Wire Line
 	3700 3750 3700 3800
@@
 	4200 3900 4200 3950
 Wire Wire Line
-	3900 3900 4050 3900
-Wire Wire Line
-	4050 3900 4200 3900
+	3900 3900 4200 3900
 Wire Wire Line
 	3900 3950 3900 3900
@@
 Connection ~ 5550 5750
 Wire Wire Line
-	4200 4350 4200 4600
-Wire Wire Line
-	4200 4600 4200 5750
-Wire Wire Line
-	3900 4350 3900 4450
-Wire Wire Line
-	3900 4450 3900 4600
-Wire Wire Line
-	3900 4600 3900 5400
+	4200 4350 4200 5750
+Wire Wire Line
+	3900 4350 3900 5400
 Wire Wire Line
 	3900 4450 5250 4450
 Wire Wire Line
-	4500 4150 4850 4150
-Wire Wire Line
-	4850 4150 5000 4150
+	4500 4150 5000 4150
 Connection ~ 6200 4150
 Connection ~ 5000 3650
@@
 Connection ~ 5550 3050
 Wire Wire Line
-	5550 3000 5550 3050
-Wire Wire Line
-	5550 3050 5550 4250
+	5550 3000 5550 4250
 Connection ~ 5550 1800
 Connection ~ 6200 1800
@@
 	5750 2350 5700 2350
 Wire Wire Line
-	5000 3600 5000 3650
-Wire Wire Line
-	5000 3650 5000 3800
+	5000 3600 5000 3800
 Wire Wire Line
 	5200 3650 5000 3650
@@
 Connection ~ 5200 2800
 Wire Wire Line
-	5200 2750 5200 2800
-Wire Wire Line
-	5200 2800 5200 2850
+	5200 2750 5200 2850
 Connection ~ 5550 2550
 Wire Wire Line
-	5500 2550 5550 2550
-Wire Wire Line
-	5550 2550 5750 2550
-Wire Wire Line
-	5550 2500 5550 2550
-Wire Wire Line
-	5550 2550 5550 2600
+	5500 2550 5750 2550
+Wire Wire Line
+	5550 2500 5550 2600
 Connection ~ 5850 4700
 Connection ~ 5550 4700
@@
 	5550 5750 5550 5700
 Wire Wire Line
-	5550 4650 5550 4700
-Wire Wire Line
-	5550 4700 5550 5400
+	5550 4650 5550 5400
 Wire Wire Line
 	7850 1900 7900 1900
@@
 	6550 5750 6550 5700
 Wire Wire Line
-	3900 5750 4200 5750
-Wire Wire Line
-	4200 5750 4550 5750
-Wire Wire Line
-	4550 5750 5550 5750
-Wire Wire Line
-	5550 5750 6550 5750
-Wire Wire Line
-	6550 5750 7200 5750
+	3900 5750 7200 5750
 Wire Wire Line
 	7200 5750 7200 2000
 Wire Wire Line
-	7200 2000 7350 2000
-Wire Wire Line
-	7350 2000 7600 2000
-Wire Wire Line
-	7600 2000 7900 2000
+	7200 2000 7900 2000
 Connection ~ 6800 1800
 Wire Wire Line
@@
 	6200 1800 6200 2850
 Wire Wire Line
-	4050 1800 4550 1800
-Wire Wire Line
-	4550 1800 5200 1800
-Wire Wire Line
-	5200 1800 5550 1800
-Wire Wire Line
-	5550 1800 6200 1800
-Wire Wire Line
-	6200 1800 6550 1800
-Wire Wire Line
-	6550 1800 6800 1800
-Wire Wire Line
-	6800 1800 7050 1800
-Wire Wire Line
-	7050 1800 7900 1800
+	4050 1800 7900 1800
 Wire Wire Line
 	6550 1800 6550 3100
 Connection ~ 6550 4150
 Wire Wire Line
-	5300 4150 6200 4150
-Wire Wire Line
-	6200 4150 6550 4150
-Wire Wire Line
-	6550 4150 7900 4150
+	5300 4150 7900 4150
 Wire Wire Line
 	6200 4500 6200 4150
@@
 	6250 4950 6200 4950
 Wire Wire Line
-	5550 4700 5850 4700
-Wire Wire Line
-	5850 4700 5900 4700
-Wire Wire Line
-	6550 4050 6550 4150
-Wire Wire Line
-	6550 4150 6550 4750
+	5550 4700 5900 4700
+Wire Wire Line
+	6550 4050 6550 4750
 Connection ~ 6200 5350
 Wire Wire Line
@@
 Connection ~ 6550 5350
 Wire Wire Line
-	5850 5350 6200 5350
-Wire Wire Line
-	6200 5350 6550 5350
+	5850 5350 6550 5350
 Wire Wire Line
 	5850 5300 5850 5350
 Wire Wire Line
-	6550 5150 6550 5350
-Wire Wire Line
-	6550 5350 6550 5400
+	6550 5150 6550 5400
 Connection ~ 6200 4950
 Wire Wire Line
-	6200 4900 6200 4950
-Wire Wire Line
-	6200 4950 6200 5000
+	6200 4900 6200 5000
 Wire Wire Line
 	5850 4700 5850 5000
@@
 Connection ~ 6550 3700
 Wire Wire Line
-	5850 3700 6200 3700
-Wire Wire Line
-	6200 3700 6550 3700
+	5850 3700 6550 3700
 Wire Wire Line
 	5850 3650 5850 3700
 Wire Wire Line
-	6550 3500 6550 3700
-Wire Wire Line
-	6550 3700 6550 3750
+	6550 3500 6550 3750
 Connection ~ 6200 3300
 Wire Wire Line
-	6200 3250 6200 3300
-Wire Wire Line
-	6200 3300 6200 3350
-Wire Wire Line
-	5550 3050 5850 3050
-Wire Wire Line
-	5850 3050 5900 3050
+	6200 3250 6200 3350
+Wire Wire Line
+	5550 3050 5900 3050
 $Comp
 L CONN_01X02 P?
@@
 	5000 2850 5000 2800
 Wire Wire Line
-	5000 2800 5200 2800
-Wire Wire Line
-	5200 2800 5250 2800
+	5000 2800 5250 2800
 $Comp
 L D D?
@@
 Connection ~ 4550 5750
 Wire Wire Line
-	4550 2500 4550 2550
-Wire Wire Line
-	4550 2550 4550 2600
+	4550 2500 4550 2600
 Wire Wire Line
 	4550 2200 4550 2150

Commit message: Add src4392i model
Parts:
- removed Q? (x5): Q_PNP_BCE, symbol Q_PNP_BCE
- removed Q?: Q_NPN_BCE, symbol Q_NPN_BCE
- added Q1, Q2, Q3, Q5, Q6: КТ313В, symbol Q_PNP_CBE
- added Q4: КТ315, symbol Q_NPN_ECB
- C18: renamed from C?; value C_Small -> 2.2k
- C19: renamed from C?; value C_Small -> 4.7
- C20: renamed from C?; value C_Small -> 100
- C21, C23: renamed from C?; value 1000.0 -> 470.0
- D2: renamed from D?; value D_Zener -> 2.7V
- D3, D4: renamed from D?; value D -> КД522А
- Q7: renamed from Q?; value Q_NPN_BCE -> КТ940А
- R15, R22: renamed from R?; value R -> 2.2k
- R16: renamed from R?; value R -> 68k
- R17: renamed from R?; value R -> 100k
- R18: renamed from R?; value R -> 470
- R19: renamed from R?; value R -> 3.3k
- R20: renamed from R?; value R -> 33k
- R21: renamed from R?; value R -> 3.9k
- R23: renamed from R?; value R -> 4.7k
- R24: renamed from R?; value R -> 4.7
- R27: renamed from R?; value R -> 47k
- RV2: renamed from RV?; value POT -> 20
- gave numbers to parts that had none: 17
Connections:
- wire segments 85 -> 86
Other:
- moved on the sheet: C18, C19, C20, C21, C22, C23, C24, D2, D3, D4, P2, P3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

Commit message: Add power
Parts:
- R15, R16, R17, R18, R19, R20, R21, R22, R23, R24, R25, R26, R27, R28, R29, R30, R31, R32: symbol R -> R-RESCUE-amplifier
- RV2: symbol POT -> POT-RESCUE-amplifier
Changed lines of the file:
@@
 EESchema Schematic File Version 2
 LIBS:amplifier-rescue
-LIBS:power
-LIBS:device
-LIBS:transistors
-LIBS:conn
-LIBS:linear
-LIBS:regul
-LIBS:74xx
-LIBS:cmos4000
-LIBS:adc-dac
-LIBS:memory
-LIBS:xilinx
-LIBS:microcontrollers
-LIBS:dsp
-LIBS:microchip
-LIBS:analog_switches
-LIBS:motorola
-LIBS:texas
-LIBS:intel
-LIBS:audio
-LIBS:interface
-LIBS:digital-audio
-LIBS:philips
-LIBS:display
-LIBS:cypress
-LIBS:siliconi
-LIBS:opto
-LIBS:atmel
-LIBS:contrib
-LIBS:valves
-LIBS:tda7293v
-LIBS:ad1955
-LIBS:src4392i
-LIBS:cdclvc1104
 LIBS:amplifier-cache
-EELAYER 26 0
+EELAYER 25 0
 EELAYER END
 $Descr A4 11693 8268
@@
 $EndDescr
 $Comp
-L R R31
+L R-RESCUE-amplifier R31
 U 1 1 588A0CB4
 P 6550 3850
@@
 $EndComp
 $Comp
-L R R32
+L R-RESCUE-amplifier R32
 U 1 1 588A0D04
 P 6550 5550
@@
 $EndComp
 $Comp
-L R R30
+L R-RESCUE-amplifier R30
 U 1 1 588A0D7E
 P 6200 5150
@@
 $EndComp
 $Comp
-L R R28
+L R-RESCUE-amplifier R28
 U 1 1 588A0DC0
 P 5850 5150
@@
 $EndComp
 $Comp
-L R R29
+L R-RESCUE-amplifier R29
 U 1 1 588A0E08
 P 6200 3450
@@
 $EndComp
 $Comp
-L R R26
+L R-RESCUE-amplifier R26
 U 1 1 588A0E99
 P 5850 3450
@@
 $EndComp
 $Comp
-L R R25
+L R-RESCUE-amplifier R25
 U 1 1 588A3B8A
 P 5550 5550
@@
 $EndComp
 $Comp
-L R R23
+L R-RESCUE-amplifier R23
 U 1 1 588A4174
 P 5200 2950
@@
 $EndComp
 $Comp
-L R R22
+L R-RESCUE-amplifier R22
 U 1 1 588A4292
 P 5000 2950
@@
 $EndComp
 $Comp
-L POT RV2
+L POT-RESCUE-amplifier RV2
 U 1 1 588A4905
 P 5550 2300
@@
 $EndComp
 $Comp
-L R R27
+L R-RESCUE-amplifier R27
 U 1 1 588A617E
 P 5850 4050
@@
 $EndComp
 $Comp
-L R R17
+L R-RESCUE-amplifier R17
 U 1 1 588A65A8
 P 3900 5550
@@
 $EndComp
 $Comp
-L R R15
+L R-RESCUE-amplifier R15
 U 1 1 588A8000
 P 3500 3350
@@
 $EndComp
 $Comp
-L R R21
+L R-RESCUE-amplifier R21
 U 1 1 588A8846
 P 4700 4650
@@
 $EndComp
 $Comp
-L R R16
+L R-RESCUE-amplifier R16
 U 1 1 588B05CD
 P 3550 4250
@@
 $EndComp
 $Comp
-L R R20
+L R-RESCUE-amplifier R20
 U 1 1 5894B398
 P 4550 2700
@@
 $EndComp
 $Comp
-L R R24
+L R-RESCUE-amplifier R24
 U 1 1 5894D3F0
 P 5550 1950
@@
 	5550 2100 5550 2150
 $Comp
-L R R18
+L R-RESCUE-amplifier R18
 U 1 1 5894EB90
 P 4050 1950
@@
 $EndComp
 $Comp
-L R R19
+L R-RESCUE-amplifier R19
 U 1 1 5894EC84
 P 4050 2950

Commit message: Update DAC
Parts:
- removed D3, D4: КД522А, symbol D
- removed R20: 33k, symbol R-RESCUE-amplifier
- added Q?: КТ313В, symbol amplifier-rescue:Q_PNP_CBE
- added R?: 68k, symbol amplifier-rescue:R-RESCUE-amplifier
- C18: value 2.2k -> 220n; symbol C_Small -> amplifier-rescue:C_Small
- C19: value 4.7 -> 1.0; symbol C_Small -> amplifier-rescue:C_Small
- C20, C22, C24: symbol C_Small -> amplifier-rescue:C_Small
- C21, C23: symbol CP_Small -> amplifier-rescue:CP_Small
- D2: symbol D_Zener -> amplifier-rescue:D_Zener
- P2, P3, P5: symbol CONN_01X02 -> amplifier-rescue:CONN_01X02
- P4: symbol CONN_01X03 -> amplifier-rescue:CONN_01X03
- Q1, Q2, Q3, Q5, Q6: symbol Q_PNP_CBE -> amplifier-rescue:Q_PNP_CBE
- Q10, Q11: symbol Q_NPN_EBC -> amplifier-rescue:Q_NPN_EBC
- Q4, Q8, Q9: symbol Q_NPN_ECB -> amplifier-rescue:Q_NPN_ECB
- Q7: symbol Q_NPN_BCE -> amplifier-rescue:Q_NPN_BCE
- R15, R18, R19, R21, R22, R23, R24, R31, R32: symbol R-RESCUE-amplifier -> amplifier-rescue:R-RESCUE-amplifier
- R16: value 68k -> 71k; symbol R-RESCUE-amplifier -> amplifier-rescue:R-RESCUE-amplifier
- R17: value 100k -> 130k; symbol R-RESCUE-amplifier -> amplifier-rescue:R-RESCUE-amplifier
- R25: value R -> 2.2k; symbol R-RESCUE-amplifier -> amplifier-rescue:R-RESCUE-amplifier
- R26, R28: value 43 -> 47; symbol R-RESCUE-amplifier -> amplifier-rescue:R-RESCUE-amplifier
- R27: value 47k -> 39k; symbol R-RESCUE-amplifier -> amplifier-rescue:R-RESCUE-amplifier
- R29, R30: value 27 -> 47; symbol R-RESCUE-amplifier -> amplifier-rescue:R-RESCUE-amplifier
- RV2: symbol POT-RESCUE-amplifier -> amplifier-rescue:POT-RESCUE-amplifier
Connections:
- net GNDPWR: now also R?.2
- net at C21.1, C22.1, P4.1 (P1)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: now also Q2.3 (E)
- net at Q2.2 (B): now also R18.2, Q?.3 (E)
- net at R19.1: now also Q?.1 (C); no longer Q2.1 (C)
- new net: Q2.1 (C), Q?.2 (B), R?.1
Other:
- moved on the sheet: C18, D2, P2, P3, Q2, R15, R16, R19
