File: DAC.sch (KiCad schematic (older format))
At the start: 83 parts

Commit message: DAC power changes
Parts:
- removed DA?: LDK220, symbol LDK220
- removed L?: 4.7uH, symbol INDUCTOR_SMALL
- added DA?: LP5900, symbol LP5900
Connections:
- net +5V: now also DA?.6 (IN)
- net +5VA: now also C?.2, DA?.1 (OUT)
- net GNDD: now also DA?.2 (N/C), DA?.3 (GND), DA?.5 (N/C)
- net at DD?.21 (CDIN/A1), DD?.24 (CDATA): now also U?.17 ((PCINT3/OC2A/MOSI)PB3); no longer U?.6 ((PCINT20/XCK/T0)PD4)
- net at DD?.25 (~CLATCH): now also U?.15 ((PCINT1/OC1A)PB1); no longer U?.3 ((PCINT17/TXD)PD1)
- net at DD?.20 (CCLK/SCL), DD?.26 (CCLK): now also U?.19 ((PCINT5/SCK)PB5); no longer U?.12 ((PCINT22/OC0A/AIN0)PD6)
- net at DD?.19 (~CS~/A0): now also U?.16 ((PCINT2/OC1B/~SS~)PB2); no longer U?.2 ((PCINT16/RXD)PD0)
- net at DD?.22 (CDOUT/SDA): now also U?.18 ((PCINT4/MISO)PB4); no longer U?.11 ((PCINT21/OC0B/T1)PD5)
- net at U?.14 ((PCINT0/CLKO/ICP1)PB0): no longer J?.2 (P2)
- net at J?.3 (P3): now also U?.24 ((PCINT9/ADC1)PC1); no longer U?.15 ((PCINT1/OC1A)PB1)
- net at J?.4 (P4): now also U?.25 ((PCINT10/ADC2)PC2); no longer U?.16 ((PCINT2/OC1B/~SS~)PB2)
- net at J?.2 (P2): now also U?.26 ((PCINT11/ADC3)PC3); no longer U?.17 ((PCINT3/OC2A/MOSI)PB3)
- net at J?.3 (P3): now also U?.27 ((PCINT12/SDA/ADC4)PC4); no longer U?.18 ((PCINT4/MISO)PB4)
- net at J?.4 (P4): now also U?.28 ((PCINT13/SCL/ADC5)PC5); no longer U?.19 ((PCINT5/SCK)PB5)
- net at U?.23 ((PCINT8/ADC0)PC0): now also J?.2 (P2)
- net at DA?.3 (EN), DA?.3 (EN), DA?.4 (EN)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: now also DA?.4 (EN)
- net at C?.1, L?.1: now also DA?.1 (OUT)
Changed lines of the file:
@@
 P 5500 2900
 F 0 "#PWR?" H 5500 2750 50  0001 C CNN
-F 1 "+1V8" H 5515 3073 50  0000 C CNN
+F 1 "+1V8" H 5500 3100 50  0000 C CNN
 F 2 "" H 5500 2900 50  0001 C CNN
 F 3 "" H 5500 2900 50  0001 C CNN
@@
 L +3V3 #PWR?
 U 1 1 5B0E6E93
-P 5950 2900
-F 0 "#PWR?" H 5950 2750 50  0001 C CNN
-F 1 "+3V3" H 5965 3073 50  0000 C CNN
-F 2 "" H 5950 2900 50  0001 C CNN
-F 3 "" H 5950 2900 50  0001 C CNN
-	1    5950 2900
+P 5650 2900
+F 0 "#PWR?" H 5650 2750 50  0001 C CNN
+F 1 "+3V3" H 5650 3050 50  0000 C CNN
+F 2 "" H 5650 2900 50  0001 C CNN
+F 3 "" H 5650 2900 50  0001 C CNN
+	1    5650 2900
 	1    0    0    -1
 $EndComp
@@
 	8300 4200 8650 4200
 Wire Wire Line
-	5650 9850 4500 9850
-Wire Wire Line
-	5650 1700 5650 9850
-Wire Wire Line
-	5650 1700 5200 1700
+	5750 9850 4500 9850
+Wire Wire Line
+	5750 1700 5750 9850
+Wire Wire Line
+	5750 1700 5200 1700
 Wire Wire Line
 	8650 4000 8400 4000
@@
 	3900 2400 3450 2400
 Wire Wire Line
-	3450 2400 3450 6500
-Wire Wire Line
 	3900 2600 3350 2600
 Wire Wire Line
-	3350 2600 3350 6600
-Wire Wire Line
-	3350 6600 6700 6600
-Wire Wire Line
-	5200 1600 5750 1600
-Wire Wire Line
-	5750 1600 5750 10150
-Wire Wire Line
 	3900 2500 3250 2500
 Wire Wire Line
-	3250 2500 3250 6700
-Wire Wire Line
-	3250 6700 6800 6700
-Wire Wire Line
-	4500 9950 5850 9950
-Wire Wire Line
-	5850 9950 5850 1500
-Wire Wire Line
-	5850 1500 5200 1500
+	4500 9950 5950 9950
+Wire Wire Line
+	5950 9950 5950 1500
+Wire Wire Line
+	5950 1500 5200 1500
 Wire Wire Line
 	1850 7700 4550 7700
 Wire Wire Line
-	4550 7700 4550 8050
-Wire Wire Line
-	4550 8050 4500 8050
-Wire Wire Line
 	1850 7600 4650 7600
 Wire Wire Line
-	4650 7600 4650 8150
-Wire Wire Line
-	4650 8150 4500 8150
-Wire Wire Line
 	1850 7500 4750 7500
 Wire Wire Line
-	4750 7500 4750 8250
-Wire Wire Line
-	4750 8250 4500 8250
-Wire Wire Line
 	1850 7400 7500 7400
 Wire Wire Line
@@
 	7450 7950 7500 7950
 Wire Wire Line
-	7450 6350 7450 9050
+	7450 6000 7450 9050
 Wire Wire Line
 	7300 8300 8850 8300
@@
 Wire Wire Line
 	8650 8050 8600 8050
-Wire Wire Line
-	4500 9750 6600 9750
-Wire Wire Line
-	3450 6500 5550 6500
-Wire Wire Line
-	5550 6500 5550 9650
-Wire Wire Line
-	5550 9650 4500 9650
-Wire Wire Line
-	5750 10150 4500 10150
-Wire Wire Line
-	6800 10250 4500 10250
 Wire Wire Line
 	8600 7950 8900 7950
@@
 	5200 3800 6000 3800
 Wire Wire Line
-	5950 3900 5200 3900
+	5650 3900 5200 3900
 Connection ~ 6800 4100
 Connection ~ 6800 3400
@@
 	7000 7650 7100 7650
 Wire Wire Line
-	5950 2900 5950 3900
-Connection ~ 5950 3800
+	5650 2900 5650 3900
+Connection ~ 5650 3800
 Connection ~ 8650 8300
 Wire Wire Line
@@
 Connection ~ 1950 7100
 Wire Wire Line
-	1850 7000 4850 7000
-Wire Wire Line
-	4850 7000 4850 8350
-Wire Wire Line
-	4850 8350 4500 8350
-Wire Wire Line
-	1850 6900 4950 6900
-Wire Wire Line
-	4950 6900 4950 8450
-Wire Wire Line
-	4950 8450 4500 8450
-Wire Wire Line
-	1850 6800 5050 6800
-Wire Wire Line
-	5050 6800 5050 8550
-Wire Wire Line
-	5050 8550 4500 8550
+	1850 7000 5350 7000
+Wire Wire Line
+	1850 6900 5450 6900
+Wire Wire Line
+	1850 6800 5550 6800
 Wire Wire Line
 	4100 5450 4050 5450
@@
 Connection ~ 7400 10700
 Wire Wire Line
-	6100 6500 5650 6500
-Connection ~ 5650 6500
+	6100 6500 5750 6500
+Connection ~ 5750 6500
 Wire Wire Line
 	6100 5500 6100 5900
@@
 Connection ~ 6100 4850
 Wire Wire Line
-	4500 9500 5450 9500
-Wire Wire Line
-	5450 9500 5450 4850
-Connection ~ 5450 4850
+	4500 9500 5650 9500
+Wire Wire Line
+	5650 9500 5650 4850
+Connection ~ 5650 4850
 Connection ~ 7000 8150
 Wire Wire Line
@@
 	8650 9450 8650 9700
 Wire Wire Line
-	8600 9350 8900 9350
+	8600 9350 9450 9350
 Wire Wire Line
 	8850 9700 8850 9650
@@
 $EndComp
 $Comp
-L LDK220 DA?
-U 1 1 5B16D3E7
-P 8050 6100
-F 0 "DA?" H 7800 6300 60  0000 C CNN
-F 1 "LDK220" H 8200 6300 60  0000 C CNN
-F 2 "" H 8100 6000 60  0001 C CNN
-F 3 "" H 8100 6000 60  0001 C CNN
-	1    8050 6100
-	1    0    0    -1
-$EndComp
-$Comp
 L C_Small C?
 U 1 1 5B16DF18
@@
 	7500 6100 6900 6100
 Connection ~ 6900 6750
-Wire Wire Line
-	7500 6000 7000 6000
-Connection ~ 7000 6000
 Wire Wire Line
 	7100 6350 7000 6350
@@
 	8850 8050 8850 7950
 Connection ~ 8850 7950
-$Comp
-L INDUCTOR_SMALL L?
-U 1 1 5B180A18
-P 9150 9350
-F 0 "L?" H 9000 9450 50  0000 C CNN
-F 1 "4.7uH" H 9250 9450 50  0000 C CNN
-F 2 "" H 9150 9350 60  0001 C CNN
-F 3 "" H 9150 9350 60  0001 C CNN
-	1    9150 9350
-	1    0    0    -1
-$EndComp
-Wire Wire Line
-	9400 9350 9450 9350
 Wire Wire Line
 	9450 9350 9450 9250
@@
 	9450 6000 9450 5900
 Wire Wire Line
-	8400 4000 8400 5450
-Wire Wire Line
-	8400 5450 6600 5450
-Wire Wire Line
-	6600 5450 6600 9750
-Wire Wire Line
 	8650 3900 8500 3900
-Wire Wire Line
-	8500 3900 8500 5550
-Wire Wire Line
-	8500 5550 6700 5550
-Wire Wire Line
-	6700 5550 6700 10050
-Wire Wire Line
-	6700 10050 4500 10050
-Connection ~ 6700 6600
-Wire Wire Line
-	6800 5650 6800 10250
-Wire Wire Line
-	6800 5650 8600 5650
-Wire Wire Line
-	8600 5650 8600 4100
-Connection ~ 6800 6700
 $Comp
 L R-RESCUE-amplifier R?
@@
 	1    0    0    -1
 $EndComp
+Wire Wire Line
+	3250 2500 3250 7300
+Wire Wire Line
+	3250 7300 6800 7300
+Wire Wire Line
+	4850 7300 4850 8550
+Wire Wire Line
+	4850 8550 4500 8550
+Wire Wire Line
+	8600 4100 8600 5700
+Wire Wire Line
+	8600 5700 6800 5700
+Wire Wire Line
+	6800 5700 6800 7300
+Connection ~ 4850 7300
+Wire Wire Line
+	8500 3900 8500 5600
+Wire Wire Line
+	8500 5600 6700 5600
+Wire Wire Line
+	3350 2600 3350 7200
+Wire Wire Line
+	3350 7200 6700 7200
+Wire Wire Line
+	6700 7200 6700 5600
+Wire Wire Line
+	4950 7200 4950 8350
+Wire Wire Line
+	4950 8350 4500 8350
+Connection ~ 4950 7200
+Wire Wire Line
+	3450 2400 3450 7100
+Wire Wire Line
+	3450 7100 5050 7100
+Wire Wire Line
+	5050 7100 5050 8250
+Wire Wire Line
+	5050 8250 4500 8250
+Wire Wire Line
+	5200 1600 5850 1600
+Wire Wire Line
+	5850 1600 5850 8450
+Wire Wire Line
+	5850 8450 4500 8450
+Wire Wire Line
+	4500 8150 6600 8150
+Wire Wire Line
+	6600 8150 6600 5500
+Wire Wire Line
+	6600 5500 8400 5500
+Wire Wire Line
+	8400 5500 8400 4000
+Wire Wire Line
+	4550 7700 4550 8900
+Wire Wire Line
+	4550 8900 4500 8900
+Wire Wire Line
+	4650 7600 4650 9000
+Wire Wire Line
+	4650 9000 4500 9000
+Wire Wire Line
+	4750 7500 4750 9100
+Wire Wire Line
+	4750 9100 4500 9100
+Wire Wire Line
+	5350 7000 5350 9200
+Wire Wire Line
+	5350 9200 4500 9200
+Wire Wire Line
+	5450 6900 5450 9300
+Wire Wire Line
+	5450 9300 4500 9300
+Wire Wire Line
+	5550 6800 5550 9400
+Wire Wire Line
+	5550 9400 4500 9400
+$Comp
+L LP5900 DA?
+U 1 1 5B20B269
+P 8050 6100
+F 0 "DA?" H 7800 6300 60  0000 C CNN
+F 1 "LP5900" H 8200 6300 60  0000 C CNN
+F 2 "" H 8050 5950 60  0001 C CNN
+F 3 "" H 8050 5950 60  0001 C CNN
+	1    8050 6100
+	1    0    0    -1
+$EndComp
+Wire Wire Line
+	8600 6200 8650 6200
+Connection ~ 8650 6200
+Wire Wire Line
+	7500 6200 7000 6200
+Connection ~ 7000 6200
+Wire Wire Line
+	7500 6000 7450 6000
 $EndSCHEMATC

Commit message: Update DAC
Parts:
- removed C? (x2): 1.0, symbol C_Small
- removed DA? (x2): LP5900, symbol LP5900
- removed DA?: LDK220, symbol LDK220
- added C?: 4.7, symbol amplifier-rescue:C_Small
- added C?: 1.0, symbol amplifier-rescue:C_Small
- added C? (x2): 470, symbol Device:C
- added C? (x8): 100, symbol Device:C
- added C? (x3): 10n, symbol Device:C
- added C? (x3): 100.0, symbol Device:CP
- added C? (x4): 560, symbol Device:C
- added C? (x4): 270, symbol Device:C
- added C? (x8): 0.1, symbol amplifier-rescue:C_Small
- added C? (x8): 47.0, symbol amplifier-rescue:CP_Small
- added DA?: LP5900, symbol amplifier-rescue:LP5900
- added DA? (x2): AD825, symbol ad825:AD825
- added DA? (x2): AD8066, symbol amplifier-rescue:AD8066
- added J?: OUT, symbol amplifier-rescue:CONN_01X03
- added L?: 4.7uH, symbol amplifier-rescue:INDUCTOR_SMALL
- added R? (x2): 33k, symbol Device:R
- added R? (x2): 100k, symbol Device:R
- added R? (x8): 2k, symbol Device:R
- added R?: 2.21k, symbol Device:R
- added R?: 2.8k, symbol Device:R
- added R? (x2): 100, symbol Device:R
- added R? (x4): 6.8k, symbol Device:R
- added R? (x4): 3.3k, symbol Device:R
- added R? (x4): 2.2k, symbol Device:R
- added R? (x4): 22, symbol Device:R
- added U? (x2): MIC5205YM5, Package_TO_SOT_SMD:SOT-23-5, symbol Regulator_Linear:MIC5205YM5
- added U?: LM317L_SO8, Package_SO:SOIC-8_3.9x4.9mm_P1.27mm, symbol Regulator_Linear:LM317L_SO8
- added U?: LM337L_SO8, Package_SO:SOIC-8_3.9x4.9mm_P1.27mm, symbol Regulator_Linear:LM337L_SO8
- C? (x26): symbol C_Small -> amplifier-rescue:C_Small
- C? (x9): symbol CP_Small -> amplifier-rescue:CP_Small
- C?: value 1.0 -> 4.7; symbol C_Small -> amplifier-rescue:C_Small
- DA? (x2): symbol LP5900 -> amplifier-rescue:LP5900
- DA?: symbol LDK220 -> amplifier-rescue:LDK220
- DA?? (x2): symbol AD8066 -> amplifier-rescue:AD8066
- DD?: symbol AD1955 -> amplifier-rescue:AD1955
- DD?: symbol SRC4392I -> amplifier-rescue:SRC4392I
- DD?? (x2): symbol KC7050 -> amplifier-rescue:KC7050
- J? (x4): symbol CONN_01X04 -> amplifier-rescue:CONN_01X04
- J?: symbol CONN_01X12 -> amplifier-rescue:CONN_01X12
- J? (x3): symbol CONN_01X05 -> amplifier-rescue:CONN_01X05
- J?: symbol CONN_01X03 -> amplifier-rescue:CONN_01X03
- JP? (x3): symbol Jumper_NC_Small -> amplifier-rescue:Jumper_NC_Small
- L? (x5): symbol INDUCTOR_SMALL -> amplifier-rescue:INDUCTOR_SMALL
- R? (x14): symbol R-RESCUE-amplifier -> amplifier-rescue:R-RESCUE-amplifier
- U?: symbol ATMEGA88A-PU -> amplifier-rescue:ATMEGA88A-PU
Connections:
- net labels added: +12VA, -12VA
- wire segments 376 -> 763
Other:
- moved on the sheet: C?, DA?, DA??A, DA??B, DD?, DD??, J?, JP?, L?, R?, U?

Commit message: Add power to DAC
Parts:
- removed U?: LM317L_SO8, Package_SO:SOIC-8_3.9x4.9mm_P1.27mm, symbol Regulator_Linear:LM317L_SO8
- removed U?: LM337L_SO8, Package_SO:SOIC-8_3.9x4.9mm_P1.27mm, symbol Regulator_Linear:LM337L_SO8
- added C52, C53: 100.0, symbol Device:CP
- added C68, C69: 1000.0, symbol Device:CP
- added C74, C75: 0.1, Capacitors_SMD:C_0805_HandSoldering, symbol Device:C
- added J10: Digital Power, symbol amplifier-rescue:CONN_01X03
- added J11: Analog Power, symbol amplifier-rescue:CONN_01X04
- added R39, R40: 3.3k, symbol Device:R
- added R43, R44: 390, symbol Device:R
- added U4: LM317_3PinPackage, symbol Regulator_Linear:LM317_3PinPackage
- added U5: LM337_SOT223, Package_TO_SOT_SMD:SOT-223-3_TabPin2, symbol Regulator_Linear:LM337_SOT223
- C10, C11, C12, C13, C14, C15, C16, C17, C19, C26, C27, C32, C33, C34, C37, C47, C50, C54, C55, C58, C59, C64, C65, C72, C73, C8, C9: renamed from C?; footprint (none) -> Capacitors_SMD:C_0805_HandSoldering
- C22, C23, C24, C25, C28, C29, C38, C39, C40, C41, C42, C43: renamed from C?; footprint (none) -> Capacitors_SMD:C_1206_HandSoldering
- gave numbers to parts that had none: 119
Connections:
- net labels added: +15V, -15V
- wire segments 763 -> 821

Commit message: Add РЭС60 footprint
Parts:
- DA7, DA8: symbol ad825:AD825 -> amplifier-rescue:AD825-ad825
Changed lines of the file:
@@
 EESchema Schematic File Version 4
-LIBS:amplifier-cache
 EELAYER 30 0
 EELAYER END
@@
 	7400 8000 7450 8000
 $Comp
-L ad825:AD825 DA7
+L amplifier-rescue:AD825-ad825 DA7
 U 1 1 5E786959
 P 13900 2200
@@
 $EndComp
 $Comp
-L ad825:AD825 DA8
+L amplifier-rescue:AD825-ad825 DA8
 U 1 1 61E0F9C1
 P 13900 4600
