File: spectrum_analyzer.sch (KiCad schematic (older format))
At the start: 178 parts, among them U7 ATmega88-20PU, U8 74145

Commit message: Add РЭС60 footprint
Parts:
- U7: symbol MCU_Microchip_ATmega:ATmega88-20PU -> amplifier-rescue:ATmega88-20PU-MCU_Microchip_ATmega
Changed lines of the file:
@@
 EESchema Schematic File Version 4
-LIBS:amplifier-cache
 EELAYER 30 0
 EELAYER END
@@
 	3300 1500 2700 1500
 $Comp
-L MCU_Microchip_ATmega:ATmega88-20PU U7
+L amplifier-rescue:ATmega88-20PU-MCU_Microchip_ATmega U7
 U 1 1 63BC476D
 P 1900 5800
@@
 	2500 5800 3000 5800
 $Comp
-L lm258:LM258 #U06
+L amplifier-rescue:LM258-lm258 #U06
 U 1 1 5DBB63B4
 P 1550 2700
@@
 $EndComp
 $Comp
-L lm258:LM258 #U06
+L amplifier-rescue:LM258-lm258 #U06
 U 2 1 5DBB7595
 P 1550 3400
