File: PowerAmplifier.sch (KiCad schematic (older format))
At the start: 42 parts, among them K1 РЭС60, P1 Filter disable, P2 INPUT, P3 POWER, P4 CLIP DETECTION, P5 OUT

Commit message: Assign footprints
Parts:
- C1, C2: footprint Capacitors_ThroughHole:CP_Radial_D8.0mm_P3.50mm -> Capacitor_THT:CP_Radial_D8.0mm_P3.50mm
- C10, C7: footprint Capacitors_ThroughHole:CP_Axial_L29.0mm_D10.0mm_P35.00mm_Horizontal -> Capacitor_THT:CP_Axial_L29.0mm_D10.0mm_P35.00mm_Horizontal
- C11, C12, C19: footprint Capacitors_ThroughHole:C_Rect_L24.0mm_W12.2mm_P22.50mm_MKT -> Capacitor_THT:C_Rect_L24.0mm_W12.2mm_P22.50mm_MKT
- C13, C16, C9: footprint Capacitors_ThroughHole:CP_Radial_D10.0mm_P2.50mm_P5.00mm -> Capacitor_THT:CP_Radial_D10.0mm_P2.50mm_P5.00mm
- C14, C15, C17: footprint Capacitors_ThroughHole:C_Rect_L18.0mm_W8.0mm_P15.00mm_FKS3_FKP3 -> Capacitor_THT:C_Rect_L18.0mm_W8.0mm_P15.00mm_FKS3_FKP3
- C18, C8: footprint Capacitors_ThroughHole:CP_Radial_D10.0mm_P5.00mm_P7.50mm -> Capacitor_THT:CP_Radial_D10.0mm_P5.00mm_P7.50mm
- C3: footprint Capacitors_ThroughHole:C_Rect_L41.5mm_W15.0mm_P37.50mm_MKS4 -> Capacitor_THT:C_Rect_L41.5mm_W15.0mm_P37.50mm_MKS4
- C4: footprint Capacitors_ThroughHole:C_Rect_L16.5mm_W9.0mm_P15.00mm_MKT -> Capacitor_THT:C_Rect_L16.5mm_W9.0mm_P15.00mm_MKT
- C5, C6: footprint Capacitors_ThroughHole:C_Rect_L16.5mm_W7.3mm_P15.00mm_MKT -> Capacitor_THT:C_Rect_L16.5mm_W7.3mm_P15.00mm_MKT
- D1, D2: footprint Diodes_ThroughHole:D_DO-15_P15.24mm_Horizontal -> Diode_THT:D_DO-15_P15.24mm_Horizontal
- DA1: footprint TO_SOT_Packages_THT:TO-220-15_Horizontal_StaggeredType1 -> Package_TO_SOT_THT:TO-220-15_P2.54x2.54mm_StaggerOdd_Lead5.84mm_TabDown
- P1, P4: footprint Pin_Headers:Pin_Header_Straight_1x02_Pitch2.54mm -> Connector_PinHeader_2.54mm:PinHeader_1x02_P2.54mm_Vertical
- P2: footprint Pin_Headers:Pin_Header_Straight_1x02_Pitch2.54mm -> Connector_PinHeader_2.54mm:PinHeader_1x03_P2.54mm_Vertical
- P3: footprint Sockets_MOLEX_KK-System:Socket_MOLEX-KK-RM3-96mm_Lock_5pin_straight -> TerminalBlock:TerminalBlock_bornier-5_P5.08mm
- P5: footprint Connect:PINHEAD1-2 -> TerminalBlock:TerminalBlock_bornier-2_P5.08mm
- R1, R10, R11, R2, R3, R4, R7, R8, R9: footprint Resistors_ThroughHole:R_Axial_DIN0207_L6.3mm_D2.5mm_P15.24mm_Horizontal -> Resistor_THT:R_Axial_DIN0309_L9.0mm_D3.2mm_P12.70mm_Horizontal
- R12: footprint Resistors_ThroughHole:R_Axial_DIN0922_L20.0mm_D9.0mm_P30.48mm_Horizontal -> Resistor_THT:R_Axial_DIN0918_L18.0mm_D9.0mm_P22.86mm_Horizontal
- R13: footprint Resistors_ThroughHole:R_Axial_Power_L25.0mm_W9.0mm_P30.48mm -> Resistor_THT:R_Axial_Power_L20.0mm_W6.4mm_P22.40mm
- R5, RV1: footprint Potentiometers:Potentiometer_Trimmer_Bourns_3296Y -> Potentiometer_THT:Potentiometer_Bourns_3296Y_Vertical
- R6: footprint Resistors_ThroughHole:R_Axial_DIN0411_L9.9mm_D3.6mm_P15.24mm_Horizontal -> Resistor_THT:R_Axial_DIN0414_L11.9mm_D4.5mm_P15.24mm_Horizontal
